File: OpenDrone_FC_F405_HW.kicad_pcb (KiCad board)
At the start: 2 copper layers, 34 x 34 mm, 90 parts, among them J1 Conn_01x05, J11 Conn_01x05, J12 Conn_01x05, J13 Conn_01x02, J14 Conn_01x02, J16 Conn_01x05, J17 Conn_02x03_Odd_Even, J2 Conn_01x02, J3 Conn_01x02, J4 Conn_01x02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

Commit message: update project
Parts:
- removed C20: 100nF, Capacitor_SMD:C_0402_1005Metric
- removed C21: 2.2nF, Capacitor_SMD:C_0402_1005Metric
- removed J13, J14, J2, J3, J4, J5, J7, J9: Conn_01x02, Footprint:HolePad_1x2
- removed J16: Conn_01x05, Footprint:Header_1x05_P2.00mm_Vertical
- removed U4: MPU6000, Footprint:QFN-24-1EP_4x4mm_P0.5mm_EP2.15x2.15mm
- added C8: 10uF, Capacitor_SMD:C_0402_1005Metric, F.Cu at (140.8, 79.3)
- added J10: Conn_01x06, Footprint:Header_1x06_P2.00mm_Vertical, F.Cu at (161.7, 74.0)
- added U3: ICM42688, Package_LGA:LGA-14_3x2.5mm_P0.5mm_LayoutBorder3x4y, F.Cu at (141.4, 83.6)
- C19: value 10nF -> 10uF
- J11, J12: value Conn_01x05 -> Conn_01x06; footprint Footprint:Header_1x05_P2.00mm_Vertical -> Footprint:Header_1x06_P2.00mm_Vertical
- moved R9 11.6 mm to (143.7, 71.8), turned to -90 degrees
- moved C19 6.74 mm to (141.8, 79.3), turned to -90 degrees
- moved C18 5.97 mm to (145.0, 83.7), turned to 180 degrees
- moved C9 2.34 mm to (145.0, 73.7), turned to 180 degrees
- moved J12 2.06 mm to (165.8, 74.0)
- moved J11 2.01 mm to (163.8, 74.0)
- moved R10 1.86 mm to (149.8, 86.2)
- moved C30 1.42 mm to (145.0, 81.8)
- moved R4 1.42 mm to (145.0, 79.9)
- moved C10 1.42 mm to (145.0, 79.0)
- moved R6 1.42 mm to (145.0, 80.9)
- moved C5 1.42 mm to (145.0, 82.7)
- moved Y2 1.38 mm to (144.2, 76.3)
- moved C28 1.26 mm to (139.9, 79.3), turned to 90 degrees
- moved C29 1.24 mm to (139.0, 79.3), turned to 90 degrees
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Connections:
- J11 pad 1: SPI2_MOSI -> unconnected-(J11-Pin_1-Pad1)
- J11 pad 2: SPI2_MISO -> I2C1_SCL
- J11 pad 3: SPI2_CLK -> I2C1_SDA
- J11 pad 4: SPI2_CS -> SPI2_CS1
- J11 pad 5: +3V3 -> SPI2_CS2
- J12 pad 1: LORA_IRQ -> unconnected-(J12-Pin_1-Pad1)
- J12 pad 2: LORA_RST -> LED_STRIP1
- J12 pad 3: I2C1_SCL -> LED_STRIP2
- J12 pad 4: I2C1_SDA -> UART4_TX
- J12 pad 5: GND -> UART4_RX
- R8 pad 1: +3V3 -> I2C2_SCL
- R8 pad 2: I2C2_SCL -> +3V3
- R9 pad 1: Net-(U4-FSYNC) -> +3V3
- R9 pad 2: GND -> Net-(U6-CSB)
- U1 pad 11: MPU6000_INT -> ICM42688_INT
- U1 pad 33: SPI2_CS -> SPI2_CS2
- U1 pad 39: unconnected-(U1-PC8-Pad39) -> SPI2_CS1
- U1 pad 44: LORA_RST -> unconnected-(U1-PA11-Pad44)
- U1 pad 45: LORA_IRQ -> unconnected-(U1-PA12-Pad45)
- U5 pad 1: MPU6000_XCL -> I2C2_SCL
- U5 pad 16: MPU6000_XDA -> I2C2_SDA
- U6 pad 2: unconnected-(U6-CSB-Pad2) -> Net-(U6-CSB)
- U6 pad 5: unconnected-(U6-SDO-Pad5) -> GND
Routing:
- net +5V: track 107.2 -> 54.2 mm
- net I2C2_SCL: track 65.5 -> 34.4 mm, vias 4 -> 3
- net I2C2_SDA: track 64.7 -> 35.3 mm, vias 4 -> 3
- net MPU6000_XDA: track 28.1 -> 0.00 mm, vias 2 -> 0
- net MPU6000_XCL: track 26.4 -> 0.00 mm, vias 2 -> 0
- net UART4_TX: track 46.7 -> 23.5 mm
- net UART4_RX: track 44.9 -> 24.0 mm
- net V_BAT: track 26.4 -> 7.20 mm
- net LORA_RST: track 14.2 -> 0.00 mm, vias 1 -> 0
- net SPI1_CLK: track 28.7 -> 15.0 mm, vias 1 -> 2
- net SPI1_CS: track 27.1 -> 14.1 mm, vias 1 -> 2
- net LORA_IRQ: track 11.7 -> 0.00 mm, vias 1 -> 0
- net ICM42688_INT: track 0.00 -> 11.2 mm, vias 0 -> 2
- net UART6_TX: track 16.3 -> 5.83 mm
- net SPI2_CS1: track 0.00 -> 9.59 mm, vias 0 -> 1
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
Commit message: update routing
Parts:
- removed D6: GREEN, LED_SMD:LED_0402_1005Metric
- removed R25: 470R, Resistor_SMD:R_0402_1005Metric
- moved C26 2.38 mm to (147.9, 67.4), turned to 90 degrees
- moved D2 1.98 mm to (149.8, 67.4)
- moved R16 1.98 mm to (148.9, 67.4)
Connections:
- U1 pad 57: LED_BLUE -> unconnected-(U1-PB5-Pad57)
Routing:
- net +5V: track 54.2 -> 67.6 mm, vias 6 -> 9
- net LED_BLUE: track 6.72 -> 0.00 mm, vias 2 -> 0
- net STM32_NRST: track 22.5 -> 17.9 mm
- net SENS_VOL: track 17.3 -> 21.1 mm
- net 5V_STEPDOWN: track 19.9 -> 23.2 mm
- net V_BAT: track 7.20 -> 9.75 mm
- net ESC1: track 14.8 -> 12.6 mm
- net ESC4: track 24.6 -> 22.7 mm
- net Net-(U5-C1): track 2.59 -> 4.37 mm
- net LED_STRIP1: track 20.9 -> 22.4 mm
- net UART4_RX: track 24.0 -> 25.3 mm
- net ESC3: track 21.3 -> 22.5 mm
- net ICM42688_INT: track 11.2 -> 12.4 mm
- net I2C1_SDA: track 16.0 -> 17.2 mm
- net 3V3_STEPDOWN: track 9.75 -> 10.9 mm
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Other:
- board text added: "LED1"
- board text added: "LED2"
- board text added: "TBD"
- board text removed: "CL2"
- board text removed: "CLK1"
- board text removed: "DA2"
- board text removed: "G"
- board text removed: "MI1"
- board text removed: "MO1"
- board text removed: "PA11"
- board text removed: "PA12"
- board text removed: "WS1"
- board text removed: "WS2"

Commit message: update routing
Parts:
- U3: footprint Package_LGA:LGA-14_3x2.5mm_P0.5mm_LayoutBorder3x4y -> Footprint:LGA-14_3x2.5mm_P0.5mm
- moved C13 0.09 mm to (166.2, 94.2), turned to 0 degrees
Connections:
- J11 pad 1: unconnected-(J11-Pin_1-Pad1) -> PC9
- J12 pad 1: unconnected-(J12-Pin_1-Pad1) -> PA8
- U1 pad 40: unconnected-(U1-PC9-Pad40) -> PC9
- U1 pad 41: unconnected-(U1-PA8-Pad41) -> PA8
Routing:
- net PA8: track 0.00 -> 22.9 mm, vias 0 -> 1
- net PC9: track 0.00 -> 10.0 mm
- net +5V: track 67.6 -> 72.0 mm, vias 9 -> 8
- net +3V3: track 126.1 -> 128.8 mm, vias 11 -> 13
- net IN_CUR: track 18.4 -> 16.3 mm
- net LED_STRIP2: track 20.7 -> 19.7 mm
- net GND: vias 68 -> 91
Other:
- board text added: "MISO2"
- board text added: "MOSI2"
- board text added: "PA8"
- board text added: "PB8"
- board text added: "PB9"
- board text added: "PC9"
- board text added: "V3.0"
- board text removed: "LED1"
- board text removed: "LED2"
- board text removed: "MI2"
- board text removed: "MO2"
- board text removed: "TBD"
- board text removed: "V2.0"

Commit message: update setting
Parts:
- J6: footprint Footprint:Connector_XH_1x08_P1.25mm_Horizontal -> KiCad-Lib:Connector_XH_1x08_P1.25mm_Horizontal
- U3: footprint Footprint:LGA-14_3x2.5mm_P0.5mm -> KiCad-Lib:LGA-14_3x2.5mm_P0.5mm
- U5: footprint Footprint:QFN-16_3x3mm_P0.5mm -> KiCad-Lib:QFN-16_3x3mm_P0.5mm
- U6: footprint Footprint:LGA-8_2x2.5mm_P0.65mm -> KiCad-Lib:LGA-8_2x2.5mm_P0.65mm
Changed lines of the file:
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@@
 		(tags "capacitor")
 		(property "Reference" "C13"
-			(at 0 -1.16 360)
+			(at 0 -1.16 0)
 			(layer "B.SilkS")
 			(hide yes)
@@
 		)
 		(property "Value" "10nF"
-			(at 0 1.16 360)
+			(at 0 1.16 0)
 			(layer "F.Fab")
 			(hide yes)
@@
 		)
 		(fp_text user "${REFERENCE}"
-			(at 0 0 360)
+			(at 0 0 0)
 			(layer "F.Fab")
 			(effects
@@
 		)
 	)
-	(footprint "Footprint:QFN-16_3x3mm_P0.5mm"
+	(footprint "KiCad-Lib:QFN-16_3x3mm_P0.5mm"
 		(layer "F.Cu")
 		(at 143.01 68.58)
 		(property "Reference" "U5"
-			(at 0 -0.5 0)
+			(at 1.78 -3.07 0)
 			(unlocked yes)
-			(layer "B.SilkS")
-			(hide yes)
+			(layer "F.SilkS")
 			(effects
 				(font
@@
 			(unlocked yes)
 			(layer "F.Fab")
-			(hide yes)
 			(effects
 				(font
@@
 			)
 		)
-		(property "Footprint" "Footprint:QFN-16_3x3mm_P0.5mm"
+		(property "Footprint" "KiCad-Lib:QFN-16_3x3mm_P0.5mm"
 			(at 0 0 0)
 			(unlocked yes)
@@
 		)
 	)
-	(footprint "Footprint:LGA-14_3x2.5mm_P0.5mm"
+	(footprint "KiCad-Lib:LGA-14_3x2.5mm_P0.5mm"
 		(layer "F.Cu")
 		(at 141.45 83.625 -90)
 		(property "Reference" "U3"
-			(at 0 -0.4 -90)
+			(at -3.43 -3.74 -90)
 			(unlocked yes)
 			(layer "F.SilkS")
@@
 			)
 		)
-		(property "Footprint" "Footprint:LGA-14_3x2.5mm_P0.5mm"
+		(property "Footprint" "KiCad-Lib:LGA-14_3x2.5mm_P0.5mm"
 			(at 0 0.09 -90)
 			(unlocked yes)
@@
 		)
 	)
-	(footprint "Footprint:Connector_XH_1x08_P1.25mm_Horizontal"
+	(footprint "KiCad-Lib:Connector_XH_1x08_P1.25mm_Horizontal"
 		(layer "F.Cu")
 		(at 136.97 91.59 90)
@@
 			(at 0 -0.5 90)
 			(unlocked yes)
-			(layer "B.SilkS")
-			(hide yes)
+			(layer "F.SilkS")
 			(effects
 				(font
@@
 			(unlocked yes)
 			(layer "F.Fab")
-			(hide yes)
 			(effects
 				(font
@@
 			)
 		)
-		(property "Footprint" "Footprint:Connector_XH_1x08_P1.25mm_Horizontal"
+		(property "Footprint" "KiCad-Lib:Connector_XH_1x08_P1.25mm_Horizontal"
 			(at 0 0 90)
 			(unlocked yes)
@@
 		)
 		(fp_text user "${REFERENCE}"
-			(at 3.62 2.39 0)
-			(unlocked yes)
+			(at 4.38 -3.8 90)
 			(layer "F.Fab")
 			(effects
@@
 		)
 		(fp_text user "${REFERENCE}"
-			(at 4.38 -3.8 90)
+			(at 0 2.5 90)
+			(unlocked yes)
 			(layer "F.Fab")
 			(effects
@@
 		)
 	)
-	(footprint "Footprint:LGA-8_2x2.5mm_P0.65mm"
+	(footprint "KiCad-Lib:LGA-8_2x2.5mm_P0.65mm"
 		(layer "F.Cu")
 		(at 140.39 75.1)
 		(property "Reference" "U6"
-			(at 0 -0.5 0)
+			(at 0.04 -2.26 0)
 			(unlocked yes)
-			(layer "B.SilkS")
-			(hide yes)
+			(layer "F.SilkS")
 			(effects
 				(font
@@
 			(unlocked yes)
 			(layer "F.Fab")
-			(hide yes)
 			(effects
 				(font
@@
 			)
 		)
-		(property "Footprint" "Footprint:LGA-8_2x2.5mm_P0.65mm"
-			(at 0 0 0)
+		(property "Footprint" "KiCad-Lib:LGA-8_2x2.5mm_P0.65mm"
+			(at -1.56 1.31 0)
 			(unlocked yes)
 			(layer "F.Fab")
@@
 		)
 		(property "Datasheet" "https://ae-bst.resource.bosch.com/media/_tech/media/datasheets/BST-BMP280-DS001.pdf"
-			(at 0 0 0)
+			(at -1.56 1.31 0)
 			(unlocked yes)
 			(layer "F.Fab")
@@
 		)
 		(property "Description" "Absolute Barometric Pressure Sensor, LGA-8"
-			(at 0 0 0)
+			(at -1.56 1.31 0)
 			(unlocked yes)
 			(layer "F.Fab")

Commit message: update
Parts:
- J1: footprint Footprint:Connector_XH_1x05_P1.25mm_Horizontal -> KiCad-Lib:Connector_XH_1x05_P1.25mm_Horizontal
- J10, J11, J12: footprint Footprint:Header_1x06_P2.00mm_Vertical -> KiCad-Lib:Header_1x06_P2.00mm_Vertical
- J8: footprint Footprint:Connector_XH_1x04_P1.25mm_Horizontal -> KiCad-Lib:Connector_XH_1x04_P1.25mm_Horizontal
- L1, L2: footprint Footprint:Inductor_SMD_4D28 -> KiCad-Lib:Inductor_SMD_4D28
- U6: footprint KiCad-Lib:LGA-8_2x2.5mm_P0.65mm -> Package_LGA:Bosch_LGA-8_2x2.5mm_P0.65mm_ClockwisePinNumbering
- U8: footprint Footprint:Board_Outline_34x34_Hole_26x26 -> Proj-Lib:Board_Outline_34x34_Hole_26x26
